File: kicad/stepper-tacho.kicad_pcb (KiCad board)
At the start: 2 copper layers, 268 x 179.1 mm, 45 parts, among them IC1 L293D, J1 IGF, J2 ILM, J3 Conn_02x03_Odd_Even, J4 STP1, J5 STP2, J6 STP4, J7 STP3, J8 ACC, J9 GND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

Commit message: first branch
Other:
- board size 268 x 179.1 mm -> 265.4 x 179.1 mm
Changed lines of the file:
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@@
     )
   )
+  (gr_line (start 16.51 15.24) (end 281.94 15.24) (angle 90) (layer Edge.Cuts) (width 0.15))
   (gr_line (start 16.51 194.31) (end 16.51 15.24) (angle 90) (layer Edge.Cuts) (width 0.15))
   (gr_line (start 281.94 194.31) (end 16.51 194.31) (angle 90) (layer Edge.Cuts) (width 0.15))
   (gr_line (start 281.94 15.24) (end 281.94 194.31) (angle 90) (layer Edge.Cuts) (width 0.15))
-  (gr_line (start 13.97 15.24) (end 281.94 15.24) (angle 90) (layer Edge.Cuts) (width 0.15))
 )
